File: controller.kicad_pcb (KiCad board)
At the start: 2 copper layers, 50.8 x 99.1 mm, 45 parts, among them J1 +12V, J2 PA, J3 PB, J4 PC, J5 UART, J6 PD, J7 VDD OUT, SW1 RESET, U1 LM317L_TO92, U2 ATmega1284-PU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

Commit message: -Improved noise filtering on supply rail (added L1 and increased C5 from 100 to 1000uF).
Parts:
- removed D1: 1N4007, Diode_THT:D_DO-41_SOD81_P2.54mm_Vertical_AnodeUp
- removed the REF** at (124.5, 48.3)
- removed the REF** at (165.1, 48.3)
- removed the REF** at (165.1, 137.2)
- removed the REF** at (124.5, 137.2)
- added L1: >=10mH, Inductor_THT:L_Toroid_Vertical_L10.0mm_W5.0mm_P5.08mm, F.Cu at (157.5, 58.4)
- added REF**: MountingHole_3.2mm_M3_Pad, MountingHole:MountingHole_3.2mm_M3_Pad, F.Cu at (165.1, 137.2)
- added REF**: MountingHole_3.2mm_M3_Pad, MountingHole:MountingHole_3.2mm_M3_Pad, F.Cu at (165.1, 48.3)
- added REF**: MountingHole_3.2mm_M3_Pad, MountingHole:MountingHole_3.2mm_M3_Pad, F.Cu at (124.5, 48.3)
- added REF**: MountingHole_3.2mm_M3_Pad, MountingHole:MountingHole_3.2mm_M3_Pad, F.Cu at (124.5, 137.2)
- C5: value 100u -> 1000u; footprint Capacitor_THT:CP_Radial_D5.0mm_P2.50mm -> Capacitor_THT:CP_Radial_D10.0mm_P2.50mm
- moved R1 7.64 mm to (162.6, 63.5)
- moved C8 6.99 mm to (149.9, 66.0), turned to 270 degrees
- moved REF** 5.08 mm to (165.1, 63.5)
- moved R2 3.97 mm to (165.1, 58.4), turned to 270 degrees
- moved J1 2.59 mm to (157.5, 48.3)
- turned C9 to 270 degrees
Connections:
- J1 pad 1: Net-(D1-Pad2) -> Net-(J1-Pad1)
- J5 pad 3: (no net) -> GND
- R1 pad 2: Net-(D1-Pad2) -> Net-(C5-Pad1)
Routing:
- net Net-(C1-Pad1): track 142.3 -> 122.3 mm
- net Net-(D1-Pad2): track 7.62 -> 0.00 mm
- net Net-(J1-Pad1): track 0.00 -> 5.08 mm
- net Net-(C5-Pad1): track 21.7 -> 24.8 mm
- net Net-(R1-Pad1): track 44.7 -> 44.2 mm
